File: hardware/relay/pcb/through_holes/relay.sch (EAGLE design)
At the start: 12 parts

Commit message: fixes in relay board
Parts:
- removed JP2: ARDUINO_POWER, SparkFun-Connectors:M02PTH
- added CN1: (no value), adafruit:DCBARRELPTH
- DEVICE, POWER: value M02PTH2 -> M025MM; device SparkFun-Connectors:M02PTH2 -> SparkFun-Connectors:M025MM
Connections:
- net GND: now also CN1.GND, CN1.GNDBREAK; no longer JP2.2
- net VCC: now also CN1.PWR; no longer JP2.1
Other:
- moved on the sheet: DEVICE, POWER
Changed lines of the file:
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@@
 <part name="C1" library="resistor" deviceset="C-EU" device="050-025X075" value="22p"/>
 <part name="C3" library="resistor" deviceset="C-EU" device="050-025X075" value="22p"/>
-<part name="JP2" library="SparkFun-Connectors" deviceset="M02" device="PTH" value="ARDUINO_POWER"/>
 <part name="C2" library="SparkFun-Passives" deviceset="CAP_POL" device="PTH1"/>
 <part name="GND1" library="supply1" deviceset="GND" device=""/>
@@
 <part name="U$1" library="SparkFun-Electromechanical" deviceset="RELAY" device="PTH"/>
 <part name="GND4" library="supply1" deviceset="GND" device=""/>
-<part name="POWER" library="SparkFun-Connectors" deviceset="M02" device="PTH2"/>
-<part name="DEVICE" library="SparkFun-Connectors" deviceset="M02" device="PTH2"/>
 <part name="D1" library="SparkFun-DiscreteSemi" deviceset="DIODE" device="1N4148"/>
+<part name="CN1" library="adafruit" deviceset="DCBARREL" device="PTH"/>
+<part name="POWER" library="SparkFun-Connectors" deviceset="M02" device="5MM"/>
+<part name="DEVICE" library="SparkFun-Connectors" deviceset="M02" device="5MM"/>
 </parts>
 <sheets>
@@
 <instance part="C1" gate="G$1" x="421.64" y="50.8"/>
 <instance part="C3" gate="G$1" x="411.48" y="55.88"/>
-<instance part="JP2" gate="G$1" x="515.62" y="106.68" rot="R180"/>
 <instance part="C2" gate="G$1" x="482.6" y="101.6"/>
 <instance part="GND1" gate="1" x="482.6" y="88.9"/>
@@
 <instance part="U$1" gate="G$1" x="426.72" y="91.44" rot="R180"/>
 <instance part="GND4" gate="1" x="441.96" y="81.28"/>
-<instance part="POWER" gate="G$1" x="378.46" y="104.14"/>
-<instance part="DEVICE" gate="G$1" x="378.46" y="78.74"/>
 <instance part="D1" gate="G$1" x="449.58" y="88.9" rot="R90"/>
+<instance part="CN1" gate="G$1" x="515.62" y="114.3"/>
+<instance part="POWER" gate="G$1" x="375.92" y="104.14"/>
+<instance part="DEVICE" gate="G$1" x="373.38" y="78.74"/>
 </instances>
 <busses>
@@
 <pinref part="C2" gate="G$1" pin="-"/>
 <pinref part="GND1" gate="1" pin="GND"/>
-<wire x1="482.6" y1="96.52" x2="482.6" y2="93.98" width="0.1524" layer="91"/>
-<pinref part="JP2" gate="G$1" pin="2"/>
-<wire x1="508" y1="104.14" x2="495.3" y2="104.14" width="0.1524" layer="91"/>
 <wire x1="495.3" y1="104.14" x2="495.3" y2="91.44" width="0.1524" layer="91"/>
 <wire x1="495.3" y1="91.44" x2="482.6" y2="91.44" width="0.1524" layer="91"/>
-<wire x1="482.6" y1="91.44" x2="482.6" y2="93.98" width="0.1524" layer="91"/>
+<wire x1="482.6" y1="91.44" x2="482.6" y2="96.52" width="0.1524" layer="91"/>
+<pinref part="CN1" gate="G$1" pin="GND"/>
+<wire x1="518.16" y1="111.76" x2="523.24" y2="111.76" width="0.1524" layer="91"/>
+<wire x1="523.24" y1="111.76" x2="523.24" y2="104.14" width="0.1524" layer="91"/>
+<wire x1="523.24" y1="104.14" x2="495.3" y2="104.14" width="0.1524" layer="91"/>
+<pinref part="CN1" gate="G$1" pin="GNDBREAK"/>
+<wire x1="518.16" y1="114.3" x2="523.24" y2="114.3" width="0.1524" layer="91"/>
+<wire x1="523.24" y1="114.3" x2="523.24" y2="111.76" width="0.1524" layer="91"/>
+<junction x="523.24" y="111.76"/>
 </segment>
 <segment>
@@
 <pinref part="C2" gate="G$1" pin="+"/>
 <wire x1="482.6" y1="104.14" x2="482.6" y2="106.68" width="0.1524" layer="91"/>
-<pinref part="JP2" gate="G$1" pin="1"/>
-<wire x1="482.6" y1="106.68" x2="508" y2="106.68" width="0.1524" layer="91"/>
+<wire x1="482.6" y1="106.68" x2="528.32" y2="106.68" width="0.1524" layer="91"/>
 <wire x1="482.6" y1="106.68" x2="419.1" y2="106.68" width="0.1524" layer="91"/>
 <junction x="482.6" y="106.68"/>
@@
 <wire x1="419.1" y1="109.22" x2="419.1" y2="106.68" width="0.1524" layer="91"/>
 <label x="431.8" y="106.68" size="1.778" layer="95"/>
+<wire x1="528.32" y1="106.68" x2="528.32" y2="116.84" width="0.1524" layer="91"/>
+<pinref part="CN1" gate="G$1" pin="PWR"/>
+<wire x1="528.32" y1="116.84" x2="518.16" y2="116.84" width="0.1524" layer="91"/>
 </segment>
 <segment>
@@
 <net name="N$7" class="0">
 <segment>
-<pinref part="POWER" gate="G$1" pin="1"/>
-<wire x1="386.08" y1="104.14" x2="411.48" y2="104.14" width="0.1524" layer="91"/>
+<wire x1="383.54" y1="104.14" x2="411.48" y2="104.14" width="0.1524" layer="91"/>
 <wire x1="411.48" y1="104.14" x2="411.48" y2="91.44" width="0.1524" layer="91"/>
 <pinref part="U$1" gate="G$1" pin="MAIN"/>
 <wire x1="411.48" y1="91.44" x2="419.1" y2="91.44" width="0.1524" layer="91"/>
+<pinref part="POWER" gate="G$1" pin="1"/>
 </segment>
 </net>
@@
 <wire x1="419.1" y1="96.52" x2="416.56" y2="96.52" width="0.1524" layer="91"/>
 <wire x1="416.56" y1="96.52" x2="416.56" y2="78.74" width="0.1524" layer="91"/>
+<wire x1="416.56" y1="78.74" x2="381" y2="78.74" width="0.1524" layer="91"/>
 <pinref part="DEVICE" gate="G$1" pin="1"/>
-<wire x1="416.56" y1="78.74" x2="386.08" y2="78.74" width="0.1524" layer="91"/>
 </segment>
 </net>
 <net name="N$9" class="0">
 <segment>
+<wire x1="391.16" y1="81.28" x2="391.16" y2="106.68" width="0.1524" layer="91"/>
+<wire x1="391.16" y1="106.68" x2="383.54" y2="106.68" width="0.1524" layer="91"/>
 <pinref part="DEVICE" gate="G$1" pin="2"/>
-<wire x1="386.08" y1="81.28" x2="391.16" y2="81.28" width="0.1524" layer="91"/>
-<wire x1="391.16" y1="81.28" x2="391.16" y2="106.68" width="0.1524" layer="91"/>
+<wire x1="381" y1="81.28" x2="391.16" y2="81.28" width="0.1524" layer="91"/>
 <pinref part="POWER" gate="G$1" pin="2"/>
-<wire x1="391.16" y1="106.68" x2="386.08" y2="106.68" width="0.1524" layer="91"/>
-</segment>
-</net>
+</segment>
+</net>
